Commit message: update

File: shelfino_description/models/shelfino_v1/xmas_hat.xacro (robot description, xacro)
@@ -2,6 +2,6 @@
 <robot name='shelfino' xmlns:xacro='http://www.ros.org/wiki/xacro'>
   <link name="shelfino${robot_id}/hat">
-    <pose>0.0 0.0 ${body_height} 0 0 0</pose>
     <visual name='visual'>
+      <origin xyz='0 0 ${body_height}' rpy='0 0 0'/>
       <geometry>
         <mesh filename='package://shelfino_description/models/xmas_hat/meshes/xmas_hat.dae' scale='0.01 0.01 0.01'/>
@@ -9,4 +9,5 @@
     </visual>
     <collision name='collision'>
+      <origin xyz='0 0 ${body_height}' rpy='0 0 0'/>
       <geometry>
         <cylinder radius='0.01' length='0.01'/>
